File: ThinkerAFE.kicad_pcb (KiCad board)
At the start: 2 copper layers, 29 x 54 mm, 57 parts, among them P1 CONN_01X10, P2 CONN_01X10, U1 TPS72325, U2 LM2664, U3 TLV70025DDC, U4 TPD4E1B06, U5 TPD4E1B06, U6 ADS1299, U7 TPD4E1B06

Commit message: laying board out
Parts:
- C1, C10, C11, C12, C13, C14, C16, C17, C2, C23, C24, C26, C27, C3, C4, C5, C6, C7, C8, C9, U1, U2: moved to B.Cu
- C36: moved to F.Cu
- moved C26 50.7 mm to (57.7, 63.8), turned to 270 degrees
- moved C27 43.7 mm to (59.3, 63.8), turned to 270 degrees
- moved C24 42.0 mm to (58.6, 59.9), turned to 180 degrees
- moved C4 27.8 mm to (42.8, 52.0)
- moved C14 26.3 mm to (47.2, 50.7), turned to 90 degrees
- moved C1 25.3 mm to (35.3, 76.9)
- moved C3 24.5 mm to (56.0, 51.2), turned to 90 degrees
- moved C13 24.4 mm to (48.8, 50.7), turned to 90 degrees
- moved U2 24.4 mm to (37.9, 76.5), turned to 270 degrees
- moved C5 23.8 mm to (42.8, 50.4)
- moved C8 23.4 mm to (36.2, 73.7), turned to 180 degrees
- moved C2 22.4 mm to (57.5, 51.2), turned to 90 degrees
- moved C10 20.4 mm to (39.2, 73.7)
- moved C7 20.3 mm to (40.5, 70.6), turned to 270 degrees
- moved C6 20.1 mm to (42.2, 70.6), turned to 270 degrees
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Routing:
- net /INSRB2: track 0.00 -> 29.0 mm, vias 0 -> 1
- net Net-(C25-Pad2): track 0.00 -> 25.4 mm
- net /IN1N: track 0.00 -> 22.8 mm, vias 0 -> 1
- net /IN2N: track 0.00 -> 20.7 mm, vias 0 -> 1
- net /IN8N: track 0.00 -> 20.2 mm, vias 0 -> 1
- net /IN3N: track 0.00 -> 18.4 mm, vias 0 -> 1
- net /IN7N: track 0.00 -> 18.0 mm, vias 0 -> 1
- net /IN4N: track 0.00 -> 16.1 mm, vias 0 -> 1
- net /IN6N: track 0.00 -> 15.9 mm, vias 0 -> 1
- net /IN5N: track 0.00 -> 15.0 mm, vias 0 -> 1
- net /6N: track 0.00 -> 7.46 mm
- net /2N: track 0.00 -> 7.11 mm
- net /8N: track 0.00 -> 6.97 mm
- net /4N: track 0.00 -> 6.90 mm
- net /BIAS: track 0.00 -> 6.80 mm
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
Commit message: Laying out the board
Parts:
- C33, C34, C35, C36, C37: moved to B.Cu
- moved C2 24.0 mm to (48.7, 73.6)
- moved C3 24.0 mm to (47.2, 73.6)
- moved C7 3.36 mm to (38.1, 68.3), turned to 180 degrees
- moved C6 2.53 mm to (41.1, 68.3), turned to 0 degrees
- moved C15 2.39 mm to (58.9, 75.4)
- moved C16 1.51 mm to (57.4, 69.9)
- moved C17 1.51 mm to (57.4, 68.3)
- moved U3 1.51 mm to (57.1, 72.7)
- moved C33 0.85 mm to (38.3, 61.3)
- moved C35 0.85 mm to (38.3, 62.9)
- moved C34 0.83 mm to (38.3, 65.1)
- moved C37 0.83 mm to (38.3, 59.7)
- moved C36 0.72 mm to (34.6, 62.5)
Routing:
- net GNDA: track 0.00 -> 26.8 mm, vias 0 -> 15
- net VDDA: track 0.00 -> 12.2 mm, vias 0 -> 4
- net VSSA: track 0.00 -> 7.93 mm, vias 0 -> 5
- net Net-(C36-Pad1): track 0.00 -> 7.25 mm, vias 0 -> 1
- net Net-(C33-Pad2): track 0.00 -> 4.64 mm, vias 0 -> 1
- net Net-(C35-Pad1): track 0.00 -> 2.80 mm, vias 0 -> 1
- added copper zone on F.Cu, net GNDA
- added copper zone on In2.Cu, net GNDA
- added copper zone on B.Cu, net VDD
- added copper zone on In1.Cu, net VDD
- added copper zone on In1.Cu, net VDDA
- added copper zone on B.Cu, net VSSA
Other:
- copper layers 2 -> 4

Commit message: Finished laying out board
Parts:
- moved C3 9.91 mm to (50.0, 64.1), turned to 180 degrees
- moved C2 8.03 mm to (50.0, 65.7), turned to 180 degrees
- moved C15 0.51 mm to (58.9, 75.9)
Routing:
- net GNDA: track 26.8 -> 66.7 mm, vias 15 -> 36
- net VDDA: track 12.2 -> 34.2 mm, vias 4 -> 13
- net VSSA: track 7.93 -> 27.6 mm, vias 5 -> 11
- net /CS: track 0.00 -> 19.1 mm, vias 0 -> 2
- net /MOSI: track 0.00 -> 16.1 mm, vias 0 -> 2
- net /SCLK: track 0.00 -> 13.9 mm, vias 0 -> 1
- net VDD: track 0.00 -> 13.9 mm, vias 0 -> 5
- net /DRDY: track 0.00 -> 13.5 mm, vias 0 -> 1
- net /MISO: track 0.00 -> 12.8 mm, vias 0 -> 1
- net /-RAW: track 0.00 -> 9.87 mm
- net Net-(C23-Pad2): track 0.00 -> 6.86 mm, vias 0 -> 1
- net Net-(C1-Pad2): track 0.00 -> 4.65 mm, vias 0 -> 2
- net Net-(C34-Pad1): track 0.00 -> 2.77 mm, vias 0 -> 1
- net Net-(C9-Pad1): track 0.00 -> 1.71 mm
- net Net-(C1-Pad1): track 0.00 -> 1.71 mm
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Other:
- rule trace_min: 0.2 -> 0.1524

Commit message: Finished layout, ready for prototyping
Parts:
- moved C2 6.88 mm to (52.9, 71.9)
- moved C3 6.88 mm to (52.9, 70.3)
- moved C34 0.09 mm to (38.3, 65.0)
Routing:
- net GNDA: track 66.7 -> 77.1 mm, vias 36 -> 34
- net VDD: track 13.9 -> 17.4 mm, vias 5 -> 6
- net Net-(C25-Pad2): track 26.6 -> 28.2 mm
- net VSSA: track 27.6 -> 26.0 mm, vias 11 -> 10
- net VDDA: track 34.2 -> 35.1 mm
Other:
- board text added: "3V3"
- board text added: "CS"
- board text added: "DRDY"
- board text added: "GND"
- board text added: "MISO"
- board text added: "MOSI"
- board text added: "Rev v0.0.1"
- board text added: "SCLK"
- board text added: "WAHO INC. 8 Channel EEG"

Commit message: saving
Parts:
- C1, C16, C17, C2, C3, C36, C6, C7, U2: moved to F.Cu
- moved C1 16.0 mm to (45.0, 64.2), turned to 180 degrees
- moved C2 15.4 mm to (56.0, 56.8), turned to 0 degrees
- moved C3 15.4 mm to (56.0, 55.3), turned to 0 degrees
- moved U2 13.9 mm to (40.7, 62.8), turned to 0 degrees
- moved C15 13.6 mm to (58.8, 62.4)
- moved P2 12.8 mm to (58.0, 67.7)
- moved C16 11.8 mm to (58.3, 58.2), turned to 90 degrees
- moved C7 11.6 mm to (35.3, 57.0)
- moved C6 11.3 mm to (35.3, 58.6), turned to 180 degrees
- moved U3 11.1 mm to (54.9, 61.8)
- moved C24 10.5 mm to (58.7, 49.4)
- moved C23 10.5 mm to (58.7, 51.0)
- moved C26 10.5 mm to (57.8, 53.3)
- moved C27 10.5 mm to (59.4, 53.3)
- moved C17 10.4 mm to (59.9, 58.2), turned to 90 degrees
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Connections:
- P2 pad 4: /SCLK -> /MISO
- P2 pad 5: /MISO -> /SCLK
- P2 pad 6: GNDA -> /CS
- P2 pad 7: /MOSI -> /RESET
- P2 pad 8: /CS -> /MOSI
- U5 pad 1: /1N -> /SRB2
- U5 pad 2: /SRB2 -> /1N
- U5 pad 4: GNDA -> Net-(U5-Pad4)
- U5 pad 5: VSSA -> Net-(U5-Pad5)
Routing:
- net GNDA: track 77.1 -> 21.9 mm, vias 34 -> 17
- net VDDA: track 35.1 -> 0.01 mm, vias 13 -> 0
- net /INSRB2: track 29.6 -> 2.19 mm, vias 3 -> 1
- net Net-(C25-Pad2): track 28.2 -> 1.71 mm, vias 2 -> 0
- net VSSA: track 26.0 -> 3.15 mm, vias 10 -> 0
- net /IN1N: track 22.8 -> 2.03 mm
- net /CS: track 19.1 -> 0.00 mm, vias 2 -> 0
- net /IN2N: track 20.7 -> 2.04 mm
- net /IN8N: track 20.2 -> 2.19 mm
- net VDD: track 17.4 -> 0.00 mm, vias 6 -> 0
- net /IN3N: track 18.4 -> 2.14 mm
- net /MOSI: track 16.1 -> 0.00 mm, vias 2 -> 0
- net /IN7N: track 18.0 -> 2.10 mm
- net /IN4N: track 16.1 -> 2.20 mm
- net /SCLK: track 13.9 -> 0.00 mm, vias 1 -> 0
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- removed copper zone on F.Cu, net GNDA
- removed copper zone on In2.Cu, net GNDA
- removed copper zone on B.Cu, net VDD
- removed copper zone on In1.Cu, net VDD
- removed copper zone on In1.Cu, net VDDA
- removed copper zone on B.Cu, net VSSA
Other:
- board size 29 x 54 mm -> 29 x 41.2 mm

Commit message: finished new layout
Parts:
- moved C3 9.90 mm to (56.7, 65.1), turned to 180 degrees
- moved C2 6.78 mm to (56.7, 63.6), turned to 180 degrees
- moved C1 4.64 mm to (40.7, 62.5), turned to 270 degrees
- moved C24 4.21 mm to (55.6, 52.2)
- moved C23 4.20 mm to (55.6, 53.8)
- moved U2 3.33 mm to (37.4, 62.0), turned to 90 degrees
- moved C16 2.99 mm to (55.9, 56.3)
- moved C17 2.49 mm to (57.5, 57.4)
- moved C7 2.27 mm to (37.6, 57.0)
- moved C6 2.26 mm to (37.6, 58.5)
Routing:
- net VDD: track 0.00 -> 19.7 mm, vias 0 -> 5
- net VDDA: track 0.01 -> 18.9 mm, vias 0 -> 13
- net GNDA: track 21.9 -> 36.3 mm, vias 17 -> 31
- net VSSA: track 3.15 -> 16.3 mm, vias 0 -> 9
- net /DRDY: track 0.00 -> 10.4 mm
- net /MOSI: track 0.00 -> 10.2 mm
- net /MISO: track 0.00 -> 10.1 mm
- net /RESET: track 0.00 -> 9.71 mm
- net /SCLK: track 0.00 -> 9.70 mm
- net /CS: track 0.00 -> 9.16 mm
- net /INSRB2: track 2.19 -> 10.7 mm
- net /-RAW: track 0.00 -> 8.03 mm, vias 0 -> 1
- net Net-(C25-Pad2): track 1.71 -> 9.42 mm
- net /IN1N: track 2.03 -> 9.25 mm
- net /IN8N: track 2.19 -> 9.03 mm
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- added copper zone on F.Cu, net GNDA
- added copper zone on In2.Cu, net GNDA
- added copper zone on B.Cu, net VDD
- added copper zone on In1.Cu, net VDDA
- added copper zone on B.Cu, net VSSA

Commit message: added text
Parts:
- C2, C3: moved to B.Cu
- moved C17 1.24 mm to (56.5, 56.7)
- moved C16 1.12 mm to (54.9, 56.7)
- moved U3 1.05 mm to (53.9, 61.9)
- moved C15 0.53 mm to (58.8, 61.9)
- moved C2 0.48 mm to (57.2, 63.6)
- moved C3 0.47 mm to (57.2, 65.2)
Routing:
- net GNDA: track 36.3 -> 40.9 mm
- net VDD: track 19.7 -> 15.5 mm
Other:
- board text added: "8 Channel EEG"
- board text added: "RESET"
- board text added: "WAHO INC."
- board text removed: "WAHO INC. 8 Channel EEG"

Commit message: Done
Routing:
- net /IN8N: track 9.03 -> 9.68 mm
- added copper zone on In1.Cu, net VDD
Other:
- board text added: "1N"
- board text added: "2N"
- board text added: "3N"
- board text added: "4N"
- board text added: "5N"
- board text added: "6N"
- board text added: "7N"
- board text added: "8N"
- board text added: "BIAS"
- board text added: "Rev v0.1.0"
- board text added: "SRB2"
- board text added: "Width: 1.15" Height: 1.62""
- board text removed: "Rev v0.0.1"
